Commit message: Refactor typography and styles across various SASS files
- Updated font sizes in _archive.scss for better readability of excerpts, meta, and citation elements.
- Adjusted heading sizes in _base.scss to improve hierarchy and consistency.
- Changed font size for custom elements in _custom.scss to align with the new typography scale.
- Modified navigation styles in _navigation.scss to utilize the new type scale for better visual coherence.
- Revised type scale definitions in _variables.scss to ensure consistent sizing across the application.
- Enhanced IK loader and robot animation scripts to include new gripper functionality and improved joint configurations.
- Added URDF configuration for UR3 robot, including detailed joint and link specifications for the Robotiq 2F-85 gripper.

File: assets/robot/ur3/ur3e.urdf (robot description, URDF)
Before this commit: robot ur3e, 8 links, 7 joints
Joints:
- joint wrist_3_link-tool0: origin xyz=0 0.09 0 rpy=0 0 0 -> xyz=0 0 0.13 rpy=0 0 0

Commit message: Refactor UR3e URDF with collision geometries and add WASM support
- Updated the UR3e URDF file to include collision geometries for each link, enhancing the kinematic model for the IK solver.
- Removed the obsolete lively_tk_lib_bg.wasm file.
- Introduced lively_bg.js, a new JavaScript file for WASM integration, providing necessary bindings and functionalities for the solver.
- Added a new lively_bg.wasm file to support the updated JavaScript functionalities.

File: assets/robot/ur3/ur3e.urdf (robot description, URDF)
Before this commit: robot ur3e, 8 links, 7 joints
Links:
- link base_link: geometry collision cylinder length=0.09 radius=0.065
- link forearm_link: geometry collision cylinder length=0.095 radius=0.04; collision cylinder length=0.20 radius=0.04
- link shoulder_link: geometry collision cylinder length=0.11 radius=0.065
- link tool0: geometry collision box size=0.09 0.09 0.13
- link upper_arm_link: geometry collision cylinder length=0.11 radius=0.04; collision cylinder length=0.11 radius=0.05
- link wrist_1_link: geometry collision cylinder length=0.095 radius=0.035
- link wrist_2_link: geometry collision cylinder length=0.1 radius=0.04
- link wrist_3_link: geometry collision cylinder length=0.04 radius=0.04
